File: projects/WaterMain/eagle/remote-connection-board.sch (EAGLE design)
At the start: 3 parts

Commit message: Added text to schematic for color coding of controll wire connection (WaterMain project)
Other:
- note added: "blue/white orange/white orange green/white green brown pair"
Changed lines of the file:
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@@
 <sheet>
 <plain>
+<text x="71.12" y="35.56" size="1.778" layer="91">blue/white
+orange/white
+orange
+green/white
+green
+brown pair</text>
 </plain>
 <instances>
@@
 </schematic>
 </drawing>
+<compatibility>
+<note version="6.3" minversion="6.2.2" severity="warning">
+Since Version 6.2.2 text objects can contain more than one line,
+which will not be processed correctly with this version.
+</note>
+</compatibility>
 </eagle>
