File: projects/PowerBlinds/eagle/motor-control-v1.brd (EAGLE design)
At the start: 40.6 x 22.9 mm, 10 parts, among them K1 351

Commit message: Added protection diode to motor control module in Power Blinds.
Parts:
- added D3: (no value), adafruit:SMADIODE
Connections:
- net N$9: now also D3.A
- net V+: now also D3.C
Changed lines of the file:
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@@
 <element name="R1" library="adafruit" package="R0603" value="2k" x="20.828" y="13.208" rot="MR270"/>
 <element name="R2" library="adafruit" package="R0603" value="300" x="27.432" y="10.414" rot="MR90"/>
+<element name="D3" library="adafruit" package="SMADIODE" value="" x="5.08" y="-5.08"/>
 </elements>
 <signals>
@@
 <wire x1="7.62" y1="14.732" x2="12.192" y2="14.732" width="0.4064" layer="16"/>
 <wire x1="12.192" y1="14.732" x2="12.827" y2="14.097" width="0.4064" layer="16"/>
+<contactref element="D3" pad="C"/>
+<wire x1="2.7305" y1="-5.08" x2="8.89" y2="7.62" width="0" layer="19" extent="1-1"/>
 </signal>
 <signal name="N$5">
@@
 <wire x1="25.0825" y1="1.778" x2="23.876" y2="1.778" width="0.8128" layer="16"/>
 <wire x1="23.876" y1="1.778" x2="22.86" y2="0.762" width="0.8128" layer="16"/>
+<contactref element="D3" pad="A"/>
+<wire x1="7.4295" y1="-5.08" x2="10.668" y2="0.762" width="0" layer="19" extent="1-16"/>
 </signal>
 <signal name="N$13">
