File: projects/PowerBlinds/eagle/motor-control-v1.sch (EAGLE design)
At the start: 10 parts, among them K1 351

Commit message: Added protection diode to motor control module in Power Blinds.
Parts:
- added D3: (no value), adafruit:DIODESMA
Connections:
- net N$9: now also D3.A
- net V+: now also D3.C
Changed lines of the file:
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@@
 <part name="P+4" library="supply1" deviceset="V+" device=""/>
 <part name="GND1" library="supply1" deviceset="GND" device=""/>
+<part name="D3" library="adafruit" deviceset="DIODE" device="SMA"/>
 </parts>
 <sheets>
@@
 <instance part="P+4" gate="1" x="-27.94" y="12.7"/>
 <instance part="GND1" gate="1" x="-27.94" y="-7.62"/>
+<instance part="D3" gate="G$1" x="25.4" y="35.56"/>
 </instances>
 <busses>
@@
 <pinref part="K1" gate="2" pin="O"/>
 <pinref part="P+1" gate="1" pin="V+"/>
-<wire x1="33.02" y1="27.94" x2="33.02" y2="38.1" width="0.1524" layer="91"/>
+<wire x1="33.02" y1="27.94" x2="33.02" y2="35.56" width="0.1524" layer="91"/>
+<pinref part="D3" gate="G$1" pin="C"/>
+<wire x1="33.02" y1="35.56" x2="33.02" y2="38.1" width="0.1524" layer="91"/>
+<wire x1="33.02" y1="35.56" x2="27.94" y2="35.56" width="0.1524" layer="91"/>
+<junction x="33.02" y="35.56"/>
 </segment>
 <segment>
@@
 <wire x1="25.4" y1="2.54" x2="20.32" y2="2.54" width="0.1524" layer="91"/>
 <junction x="20.32" y="2.54"/>
+<pinref part="D3" gate="G$1" pin="A"/>
+<wire x1="22.86" y1="35.56" x2="20.32" y2="35.56" width="0.1524" layer="91"/>
+<wire x1="20.32" y1="35.56" x2="20.32" y2="27.94" width="0.1524" layer="91"/>
+<junction x="20.32" y="27.94"/>
 </segment>
 </net>
